File: var_rename_test.kicad_sch (KiCad schematic)
At the start: 1 part

Commit message: trying with footprint in user lib
Parts:
- R1: footprint TestPoint:TestPoint_Bridge_Pitch2.0mm_Drill0.7mm -> var_rename:D_0805_2012Metric; left:Footprint Resistor_SMD:R_0805_2012Metric -> var_rename:D_0805_2012Metric; right:Footprint TestPoint:TestPoint_Bridge_Pitch2.0mm_Drill0.7mm -> var_rename:TestPoint_Bridge_Pitch2.0mm_Drill0.7mm
Changed lines of the file:
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@@
       (effects (font (size 1.27 1.27)) (justify left))
     )
-    (property "Footprint" "TestPoint:TestPoint_Bridge_Pitch2.0mm_Drill0.7mm" (at 141.732 78.74 90)
+    (property "Footprint" "var_rename:D_0805_2012Metric" (at 141.732 78.74 90)
       (effects (font (size 1.27 1.27)) (hide yes))
     )
@@
       (effects (font (size 1.27 1.27)) (hide yes))
     )
-    (property "left:Footprint" "Resistor_SMD:R_0805_2012Metric" (at 143.51 78.74 0)
+    (property "left:Footprint" "var_rename:D_0805_2012Metric" (at 143.51 78.74 0)
       (effects (font (size 1.27 1.27)) (hide yes))
     )
-    (property "right:Footprint" "TestPoint:TestPoint_Bridge_Pitch2.0mm_Drill0.7mm" (at 143.51 78.74 0)
+    (property "right:Footprint" "var_rename:TestPoint_Bridge_Pitch2.0mm_Drill0.7mm" (at 143.51 78.74 0)
       (effects (font (size 1.27 1.27)) (hide yes))
     )
